File: hardware/schematic.sch (EAGLE design)
At the start: 94 parts, among them IC1 STM8S005K6T6C, IC2 78L05F, IC3 TLC272D, Q1 J3Y, Q2 Si2300DS, Q3 J3Y, Q4 IRFP150N, Q5 J3Y, U1 TL431PTH, Y1 10M

Commit message: Schematic: Added Displayboard; Readme: Added Image
Parts:
- added C29, C30: 100nF, SparkFun-Capacitors:CAP0805
- added DP1_DIG1, DP1_DIG2, DP1_DIG3, DP1_DIG4, DP2_DIG1, DP2_DIG2, DP2_DIG3: 7-SEGMENT-DISPLAY-1"-RED, SparkFun-Displays:7-SEGMENT-DISPLAY-1"-RED
- added D_A, D_AH, D_HIGH, D_LOW, D_RUN, D_V, D_WH: (no value), SparkFun-LED:LED3MM
- added IC4, IC5: TM1650_SOP, rgb_matrix:TM1650_SOP
- added JP8: DISP, SparkFun-Connectors:M10SILK_FEMALE_PTH
- added R41, R42: 5k1, SparkFun-Resistors:RESISTOR0805-RES
- added S1: OK, SparkFun-Electromechanical:SWITCH-MOMENTARY-4_PTH
- added SW1: ROTARTY_ENCODER, SparkFun-Electromechanical:ROTARTY_ENCODER
Connections:
- new net DP1: DP1_DIG1.A, DP1_DIG1.B, DP1_DIG1.C, DP1_DIG1.D, DP1_DIG1.DP, DP1_DIG1.E, DP1_DIG1.F, DP1_DIG1.G, DP1_DIG1.G1, DP1_DIG1.G2, DP1_DIG2.A, DP1_DIG2.B, DP1_DIG2.C, DP1_DIG2.D, DP1_DIG2.DP, DP1_DIG2.E, DP1_DIG2.F, DP1_DIG2.G, DP1_DIG2.G1, DP1_DIG2.G2, DP1_DIG3.A, DP1_DIG3.B, DP1_DIG3.C, DP1_DIG3.D, DP1_DIG3.DP, DP1_DIG3.E, DP1_DIG3.F, DP1_DIG3.G, DP1_DIG3.G1, DP1_DIG3.G2, DP1_DIG4.A, DP1_DIG4.B, DP1_DIG4.C, DP1_DIG4.D, DP1_DIG4.DP, DP1_DIG4.E, DP1_DIG4.F, DP1_DIG4.G, DP1_DIG4.G1, DP1_DIG4.G2, IC4.A, IC4.B, IC4.C, IC4.D, IC4.DIG1, IC4.DIG2, IC4.DIG3, IC4.DIG4, IC4.E, IC4.F, IC4.G, IC4.KP
- new net DP2: DP2_DIG1.A, DP2_DIG1.B, DP2_DIG1.C, DP2_DIG1.D, DP2_DIG1.DP, DP2_DIG1.E, DP2_DIG1.F, DP2_DIG1.G, DP2_DIG1.G1, DP2_DIG1.G2, DP2_DIG2.A, DP2_DIG2.B, DP2_DIG2.C, DP2_DIG2.D, DP2_DIG2.DP, DP2_DIG2.E, DP2_DIG2.F, DP2_DIG2.G, DP2_DIG2.G1, DP2_DIG2.G2, DP2_DIG3.A, DP2_DIG3.B, DP2_DIG3.C, DP2_DIG3.D, DP2_DIG3.DP, DP2_DIG3.E, DP2_DIG3.F, DP2_DIG3.G, DP2_DIG3.G1, DP2_DIG3.G2, D_A.A, D_A.C, D_AH.A, D_AH.C, D_HIGH.A, D_HIGH.C, D_LOW.A, D_LOW.C, D_RUN.A, D_RUN.C, D_V.A, D_V.C, D_WH.A, D_WH.C, IC5.A, IC5.B, IC5.C, IC5.D, IC5.DIG1, IC5.DIG2, IC5.DIG3, IC5.DIG4, IC5.E, IC5.F, IC5.G, IC5.KP
- new net ENC_A_DP: JP8.10, SW1.A
- new net ENC_B_DP: JP8.9, SW1.B
- new net ENC_P_DP: JP8.7, SW1.SW+
- new net GND-ISO: C29.2, C30.2, IC4.GND, IC5.GND, JP8.1, JP8.2, S1.3, S1.4, SW1.C, SW1.SW-
- new net RUN_P_DP: JP8.8, S1.1, S1.2
- new net SCL_DP: IC4.SCL, IC5.SCL, JP8.6
- new net SDA1_DP: IC5.SDA, JP8.5, R42.2
- new net SDA2_DP: IC4.SDA, JP8.4, R41.2
- new net VCC-ISO: C29.1, C30.1, IC4.VDD, IC5.VDD, JP8.3, R41.1, R42.1
Other:
- note added: "A"
- note added: "B"
- note added: "Bottom Display"
- note added: "C"
- note added: "D"
- note added: "DIG1"
- note added: "DIG2"
- note added: "DIG3"
- note added: "DIG4"
- note added: "Display Connector"
- note added: "E"
- note added: "F"
- note added: "G"
- note added: "Inputs"
- note added: "Top Display"
